File: trackpad.kicad_sch (KiCad schematic)
At the start: 4 parts, among them J7 Conn_02x10_Odd_Even_MountingP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

Commit message: trackpad
Parts:
- removed C6: 0.1uF, Capacitor_SMD:C_0603_1608Metric, symbol Device:C_Small
- removed J7: Conn_02x10_Odd_Even_MountingPin, keeb-libs:hirose-df30fb-20ds-0.4v(82), symbol Connector_Generic_MountingPin:Conn_02x10_Odd_Even_MountingPin
- removed R11, R4: 220k, Resistor_SMD:R_0603_1608Metric, symbol Device:R
Connections:
- no-connect marks 7 -> 0
Changed lines of the file:
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@@
 (kicad_sch (version 20210621) (generator eeschema)
   (paper "A4")
-  (junction (at 128.27 114.3) (diameter 1.016) (color 0 0 0 0))
-  (no_connect (at 119.38 88.9))
-  (no_connect (at 132.08 86.36))
-  (no_connect (at 132.08 88.9))
-  (no_connect (at 132.08 91.44))
-  (no_connect (at 132.08 93.98))
-  (no_connect (at 132.08 104.14))
-  (no_connect (at 132.08 106.68))
-  (wire (pts (xy 119.38 118.11) (xy 119.38 109.22))
-    (stroke (width 0) (type solid) (color 0 0 0 0))
-  )
-  (wire (pts (xy 123.19 118.11) (xy 119.38 118.11))
-    (stroke (width 0) (type solid) (color 0 0 0 0))
-  )
-  (wire (pts (xy 128.27 114.3) (xy 125.73 114.3))
-    (stroke (width 0) (type solid) (color 0 0 0 0))
-  )
-  (wire (pts (xy 128.27 114.3) (xy 128.27 118.11))
-    (stroke (width 0) (type solid) (color 0 0 0 0))
-  )
-  (wire (pts (xy 132.08 99.06) (xy 139.7 99.06))
-    (stroke (width 0) (type solid) (color 0 0 0 0))
-  )
-  (wire (pts (xy 132.08 109.22) (xy 132.08 114.3))
-    (stroke (width 0) (type solid) (color 0 0 0 0))
-  )
-  (wire (pts (xy 132.08 114.3) (xy 128.27 114.3))
-    (stroke (width 0) (type solid) (color 0 0 0 0))
-  )
-  (wire (pts (xy 139.7 99.06) (xy 139.7 96.52))
-    (stroke (width 0) (type solid) (color 0 0 0 0))
-  )
-  (hierarchical_label "GND" (shape input) (at 119.38 86.36 180)
-    (effects (font (size 1.27 1.27)) (justify right))
-  )
-  (hierarchical_label "RST_2V8" (shape input) (at 119.38 91.44 180)
-    (effects (font (size 1.27 1.27)) (justify right))
-  )
-  (hierarchical_label "SHTDWN_2V8" (shape input) (at 119.38 93.98 180)
-    (effects (font (size 1.27 1.27)) (justify right))
-  )
-  (hierarchical_label "~{CS}_2V8" (shape input) (at 119.38 96.52 180)
-    (effects (font (size 1.27 1.27)) (justify right))
-  )
-  (hierarchical_label "SCK_2V8" (shape input) (at 119.38 99.06 180)
-    (effects (font (size 1.27 1.27)) (justify right))
-  )
-  (hierarchical_label "MOSI_2V8" (shape input) (at 119.38 101.6 180)
-    (effects (font (size 1.27 1.27)) (justify right))
-  )
-  (hierarchical_label "MISO_2V8" (shape output) (at 119.38 104.14 180)
-    (effects (font (size 1.27 1.27)) (justify right))
-  )
-  (hierarchical_label "MOTION_2V8" (shape output) (at 119.38 106.68 180)
-    (effects (font (size 1.27 1.27)) (justify right))
-  )
-  (hierarchical_label "2V8" (shape input) (at 119.38 109.22 180)
-    (effects (font (size 1.27 1.27)) (justify right))
-  )
-  (hierarchical_label "GND" (shape input) (at 132.08 109.22 0)
-    (effects (font (size 1.27 1.27)) (justify left))
-  )
-  (hierarchical_label "2V8" (shape input) (at 139.7 99.06 0)
-    (effects (font (size 1.27 1.27)) (justify left))
-  )
-  (hierarchical_label "GND" (shape input) (at 139.7 101.6 0)
-    (effects (font (size 1.27 1.27)) (justify left))
-  )
-  (symbol (lib_id "Device:R") (at 135.89 96.52 90) (unit 1)
-    (in_bom yes) (on_board yes)
-    (property "Reference" "R4" (id 0) (at 135.89 94.0774 90))
-    (property "Value" "220k" (id 1) (at 135.89 96.8525 90))
-    (property "Footprint" "Resistor_SMD:R_0603_1608Metric" (id 2) (at 135.89 98.298 90)
-      (effects (font (size 1.27 1.27)) hide)
-    )
-    (property "Datasheet" "~" (id 3) (at 135.89 96.52 0)
-      (effects (font (size 1.27 1.27)) hide)
-    )
-    (pin "1")
-    (pin "2")
-  )
-  (symbol (lib_id "Device:R") (at 135.89 101.6 90) (unit 1)
-    (in_bom yes) (on_board yes)
-    (property "Reference" "R11" (id 0) (at 135.89 104.2374 90))
-    (property "Value" "220k" (id 1) (at 135.89 101.9325 90))
-    (property "Footprint" "Resistor_SMD:R_0603_1608Metric" (id 2) (at 135.89 103.378 90)
-      (effects (font (size 1.27 1.27)) hide)
-    )
-    (property "Datasheet" "~" (id 3) (at 135.89 101.6 0)
-      (effects (font (size 1.27 1.27)) hide)
-    )
-    (pin "1")
-    (pin "2")
-  )
-  (symbol (lib_id "Device:C_Small") (at 125.73 118.11 90) (unit 1)
-    (in_bom yes) (on_board yes)
-    (property "Reference" "C6" (id 0) (at 125.73 121.4713 90))
-    (property "Value" "0.1uF" (id 1) (at 125.73 122.9764 90))
-    (property "Footprint" "Capacitor_SMD:C_0603_1608Metric" (id 2) (at 125.73 118.11 0)
-      (effects (font (size 1.27 1.27)) hide)
-    )
-    (property "Datasheet" "~" (id 3) (at 125.73 118.11 0)
-      (effects (font (size 1.27 1.27)) hide)
-    )
-    (pin "1")
-    (pin "2")
-  )
-  (symbol (lib_id "Connector_Generic_MountingPin:Conn_02x10_Odd_Even_MountingPin") (at 124.46 96.52 0) (unit 1)
-    (in_bom yes) (on_board yes) (fields_autoplaced)
-    (property "Reference" "J7" (id 0) (at 125.73 81.1234 0))
-    (property "Value" "Conn_02x10_Odd_Even_MountingPin" (id 1) (at 125.73 83.8985 0))
-    (property "Footprint" "keeb-libs:hirose-df30fb-20ds-0.4v(82)" (id 2) (at 124.46 96.52 0)
-      (effects (font (size 1.27 1.27)) hide)
-    )
-    (property "Datasheet" "~" (id 3) (at 124.46 96.52 0)
-      (effects (font (size 1.27 1.27)) hide)
-    )
-    (pin "1")
-    (pin "10")
-    (pin "11")
-    (pin "12")
-    (pin "13")
-    (pin "14")
-    (pin "15")
-    (pin "16")
-    (pin "17")
-    (pin "18")
-    (pin "19")
-    (pin "2")
-    (pin "20")
-    (pin "3")
-    (pin "4")
-    (pin "5")
-    (pin "6")
-    (pin "7")
-    (pin "8")
-    (pin "9")
-    (pin "MP")
-  )
 )
