File: trackpad_conn.kicad_sch (KiCad schematic)
At the start: 7 parts, among them U6 MIC5365-2.8YC5, U7 4050

Commit message: trackpad
Parts:
- added C6: 0.1uF, Capacitor_SMD:C_0603_1608Metric, symbol Device:C_Small
- added J5: Conn_02x10_Odd_Even_MountingPin, keeb-libs:hirose-df30fb-20ds-0.4v(82), symbol Connector_Generic_MountingPin:Conn_02x10_Odd_Even_MountingPin
- added R11, R4: 220k, Resistor_SMD:R_0603_1608Metric, symbol Device:R
Connections:
- net +2V8: now also C6.1, J5.12 (Pin_12), J5.19 (Pin_19), R4.2
- net GND: now also C6.2, J5.1 (Pin_1), J5.20 (Pin_20), J5.MP (MountPin), R11.2
- net MOSI_2V8: now also J5.13 (Pin_13)
- net SCK_2V8: now also J5.11 (Pin_11)
- net SHTDWN_2V8: now also J5.7 (Pin_7)
- net ~{CS}_2V8: now also J5.9 (Pin_9)
- new net MISO_2V8: J5.15 (Pin_15)
- new net MOTION_2V8: J5.17 (Pin_17)
- new net R11_conn: J5.14 (Pin_14), R11.1
- new net R4_conn: J5.10 (Pin_10), R4.1
- new net RST_2V8: J5.5 (Pin_5)
- no-connect marks 0 -> 7
