File: fusion.kicad_pcb (KiCad board)
At the start: 2 copper layers, 278.9 x 113.3 mm, 68 parts, among them J1 Conn_01x04_Female, J2 USB_C_Receptacle_USB2.0, J3 Conn_02x10_Odd_Even, J4 Conn_02x10_Odd_Even, K1 KEY, K10 KEY, K11 KEY, K12 KEY, K13 KEY, K14 KEY, K15 KEY, K16 KEY, K17 KEY, K18 KEY, K19 KEY, K2 KEY, K20 KEY, K21 KEY, K22 KEY, K23 KEY, K24 KEY, K25 KEY, K26 KEY, K27 KEY, K28 KEY, K29 KEY, K3 KEY, K30 KEY, K31 KEY, K32 KEY, K33 KEY, K34 KEY, K35 KEY, K36 KEY, K37 KEY, K38 KEY, K4 KEY, K5 KEY, K6 KEY, K7 KEY, K8 KEY, K9 KEY, SW1 SW_Push, U1 Holyiot_18010, U2 MT25QL128ABA1ESE, U3 BQ24075, U4 XC6220B331MR, U5 LN4913

Commit message: fpc and hinges
Parts:
- removed the REF** at (155.5, 160.0)
- added REF**: hinge-conn-2, fusion:hinge-conn-2, F.Cu at (141.5, 77.1)
- added REF**: hinge, fusion:hinge, F.Cu at (139.0, 147.4)
- added REF**: hinge-conn-1, fusion:hinge-conn-1, F.Cu at (141.5, 121.6)
- added REF**: hinge-conn-1, fusion:hinge-conn-1, F.Cu at (140.5, 77.1)
- added REF**: hinge-conn-2, fusion:hinge-conn-2, F.Cu at (140.5, 121.6)
- J3, J4: value Conn_02x10_Odd_Even -> Conn_01x22; footprint Connector_PinHeader_1.27mm:PinHeader_2x10_P1.27mm_Vertical_SMD -> Connector_FFC-FPC:Hirose_FH12-22S-0.5SH_1x22-1MP_P0.50mm_Horizontal
- moved BT1 25.8 mm to (114.8, 70.4)
- moved J4 3.25 mm to (160.8, 85.9), turned to -90 degrees
- moved R5 2.82 mm to (163.2, 77.1)
- moved R8 2.82 mm to (163.2, 75.6)
- moved C1 2.82 mm to (163.2, 74.1)
- moved K18 2.68 mm to (102.3, 140.1)
- moved K1 2.68 mm to (30.7, 82.6)
- moved K10 2.68 mm to (98.6, 94.1)
- moved K11 2.68 mm to (25.9, 109.3)
- moved K12 2.68 mm to (45.9, 95.5)
- moved K13 2.68 mm to (65.1, 93.4)
- moved K14 2.68 mm to (80.7, 104.8)
- moved K15 2.68 mm to (95.1, 107.1)
- moved K16 2.68 mm to (74.6, 127.5)
- moved K2 2.68 mm to (53.7, 66.5)
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Connections:
- J3 pad 1: L_BAT -> L_K18
- J3 pad 10: L_K8 -> L_K7
- J3 pad 11: L_K7 -> L_K8
- J3 pad 12: L_K6 -> L_K9
- J3 pad 13: L_K15 -> L_K10
- J3 pad 14: L_K14 -> L_K1
- J3 pad 15: L_K13 -> L_K2
- J3 pad 16: L_K12 -> L_K3
- J3 pad 17: L_K11 -> L_K4
- J3 pad 18: L_K16 -> L_K5
- J3 pad 19: L_K17 -> L_GND
- J3 pad 2: L_GND -> L_K17
- J3 pad 20: L_K18 -> L_GND
- J3 pad 3: L_K5 -> L_K16
- J3 pad 4: L_K4 -> L_K11
- J3 pad 5: L_K3 -> L_K12
- J3 pad 6: L_K2 -> L_K13
- J3 pad 7: L_K1 -> L_K14
- J3 pad 8: L_K10 -> L_K15
- J3 pad 9: L_K9 -> L_K6
- J4 pad 1: GND -> BAT
- J4 pad 10: K8 -> K10
- J4 pad 11: K7 -> K9
- J4 pad 12: K6 -> K8
- J4 pad 13: K15 -> K7
- J4 pad 14: K14 -> K6
- J4 pad 15: K13 -> K15
- J4 pad 16: K12 -> K14
- J4 pad 17: K11 -> K13
- J4 pad 18: K16 -> K12
- J4 pad 19: K17 -> K11
- J4 pad 20: K18 -> K16
- J4 pad 3: K5 -> GND
- J4 pad 4: K4 -> GND
- J4 pad 5: K3 -> K5
- J4 pad 6: K2 -> K4
- J4 pad 7: K1 -> K3
- J4 pad 8: K10 -> K2
- J4 pad 9: K9 -> K1
- U1 pad 31: K18 -> K17
- U1 pad 43: K17 -> K18
Routing:
- net L_BAT: track 38.6 -> 13.6 mm
- net L_GND: track 383.0 -> 361.2 mm, vias 1 -> 0
- net L_K2: track 95.3 -> 84.3 mm, vias 2 -> 0
- net L_K18: track 69.0 -> 58.8 mm, vias 2 -> 0
- net L_K4: track 53.6 -> 43.4 mm, vias 2 -> 0
- net L_K10: track 49.6 -> 39.5 mm, vias 2 -> 0
- net L_K8: track 86.2 -> 76.2 mm, vias 2 -> 0
- net L_K14: track 79.9 -> 70.0 mm, vias 2 -> 0
- net L_K6: track 142.5 -> 132.6 mm, vias 2 -> 0
- net L_K12: track 117.4 -> 107.6 mm, vias 2 -> 0
- net L_K16: track 84.6 -> 75.0 mm, vias 2 -> 0
- net GND: track 473.3 -> 481.9 mm, vias 15 -> 17
- net K17: track 5.95 -> 11.8 mm, vias 0 -> 1
- net BAT: track 19.5 -> 24.4 mm
- net K9: track 12.9 -> 16.6 mm
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Other:
- board size 278.9 x 113.3 mm -> 276.3 x 95.6 mm

Commit message: bug
Parts:
- removed D2: RED, LED_SMD:LED_0805_2012Metric
- removed the REF** at (141.5, 77.1)
- removed the REF** at (139.0, 147.4)
- removed the REF** at (141.5, 121.6)
- removed the REF** at (140.5, 77.1)
- removed the REF** at (140.5, 121.6)
- added C6: 0.1uF, Capacitor_SMD:C_0603_1608Metric, F.Cu at (89.3, 87.9)
- added D1: RED, LED_SMD:LED_0805_2012Metric, F.Cu at (190.3, 102.8)
- added J5: trackpad, fusion:trackpad, F.Cu at (94.7, 92.3)
- added J6: trackpad_conn, fusion:trackpad_conn, F.Cu at (233.2, 170.0)
- added J7: Conn_02x10_Odd_Even_MountingPin, keeb-libs:hirose-df30fb-20ds-0.4v(82), F.Cu at (87.1, 83.5)
- added JP2: SolderJumper_2_Open, Jumper:SolderJumper-2_P1.3mm_Open_RoundedPad1.0x1.5mm, F.Cu at (239.9, 165.0)
- added JP3: SolderJumper_2_Open, Jumper:SolderJumper-2_P1.3mm_Open_RoundedPad1.0x1.5mm, F.Cu at (240.8, 168.3)
- added JP4: SolderJumper_2_Open, Jumper:SolderJumper-2_P1.3mm_Open_RoundedPad1.0x1.5mm, F.Cu at (241.7, 171.6)
- added JP5: SolderJumper_2_Open, Jumper:SolderJumper-2_P1.3mm_Open_RoundedPad1.0x1.5mm, F.Cu at (253.2, 169.0)
- added JP6: Jumper_3_Open, Jumper:SolderJumper-3_P2.0mm_Open_TrianglePad1.0x1.5mm_NumberLabels, F.Cu at (184.3, 114.0)
- added R11: 220k, Resistor_SMD:R_0603_1608Metric, F.Cu at (82.3, 85.6)
- added R4: 220k, Resistor_SMD:R_0603_1608Metric, F.Cu at (82.3, 82.6)
- added REF**: hinge-conn-2, fusion:hinge-conn-2, F.Cu at (157.5, 121.9)
- added REF**: hinge-conn-1, fusion:hinge-conn-1, F.Cu at (157.5, 166.5)
- added REF**: magnet-fp, fusion:magnet-fp, F.Cu at (-84.1, 86.9)
- added REF**: trackpad-hole, fusion:trackpad-hole, F.Cu at (69.7, 94.3)
- added REF**: hinge-conn-1, fusion:hinge-conn-1, F.Cu at (26.1, 98.7)
- added REF**: hinge-conn-2, fusion:hinge-conn-2, F.Cu at (26.1, 143.3)
- added U6: MIC5365-2.8YC5, Package_TO_SOT_SMD:SOT-353_SC-70-5, F.Cu at (239.4, 160.9)
- added U7: 4050, Package_SO:SOIC-16_3.9x9.9mm_P1.27mm, F.Cu at (246.6, 166.8)
- J3, J4: value Conn_01x22 -> Conn_01x12_MountingPin; footprint Connector_FFC-FPC:Hirose_FH12-22S-0.5SH_1x22-1MP_P0.50mm_Horizontal -> Connector_FFC-FPC:Hirose_FH12-12S-0.5SH_1x12-1MP_P0.50mm_Horizontal
- JP1: value Jumper_3_Open -> SolderJumper_2_Open; footprint Jumper:SolderJumper-3_P2.0mm_Open_TrianglePad1.0x1.5mm_NumberLabels -> Jumper:SolderJumper-2_P1.3mm_Open_RoundedPad1.0x1.5mm
- K1, K10, K11, K15, K37, K38, K5, K6: value KEY -> diode-choc; footprint keeb-libs:pg1232-shorter-right -> pg1232:pg1232-DSSR
- K12, K13, K16, K17, K18, K2, K21, K22, K26, K27, K3, K31, K32, K34, K35, K36, K7, K8: value KEY -> diode-choc; footprint keeb-libs:pg1232-short -> pg1232:pg1232-DSS
- K14, K4, K9: value KEY -> diode-choc; footprint keeb-libs:pg1232-short-left -> pg1232:pg1232-DSSL
- K19, K23, K24, K28, K29, K33: value KEY -> diode-choc; footprint keeb-libs:pg1232-shorter-left -> pg1232:pg1232-DSSL
- K20, K25, K30: value KEY -> diode-choc; footprint keeb-libs:pg1232-short-right -> pg1232:pg1232-DSSR
- moved K18 121.5 mm to (-17.7, 159.5)
- moved JP1 120.6 mm to (243.3, 159.8), turned to -75 degrees
- moved K17 120.4 mm to (-30.1, 153.6)
- moved K16 119.2 mm to (-42.7, 148.7)
- moved BT1 116.4 mm to (0.31, 91.8)
- moved K3 115.2 mm to (-40.8, 83.1)
- moved K4 115.2 mm to (-25.2, 94.5)
- moved K2 115.2 mm to (-60.0, 85.2)
- moved K1 114.6 mm to (-82.6, 99.8)
- moved K10 114.6 mm to (-14.7, 111.3)
- moved K15 114.6 mm to (-18.2, 124.3)
- moved K7 114.6 mm to (-63.5, 98.2)
- moved K9 114.6 mm to (-28.7, 107.5)
- moved K6 114.6 mm to (-86.1, 112.9)
- moved K8 114.6 mm to (-44.3, 96.1)
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Connections:
- net DISP_CS renamed DISP_~{CS}
- net FLASH_CS renamed FLASH_~{CS}
- net ~{CHG} renamed Net-(R6-Pad1)
- BT1 pad 1: L_BAT -> /left/BAT
- BT1 pad 2: L_GND -> /left/GND
- J3 pad 1: L_K18 -> /left/BAT
- J3 pad 10: L_K7 -> /left/C2
- J3 pad 11: L_K8 -> /left/C1
- J3 pad 12: L_K9 -> /left/C0
- J3 pad 2: L_K17 -> /left/GND
- J3 pad 3: L_K16 -> unconnected-(J3-Pad3)
- J3 pad 4: L_K11 -> /left/R3
- J3 pad 5: L_K12 -> /left/R2
- J3 pad 6: L_K13 -> /left/R1
- J3 pad 7: L_K14 -> /left/R0
- J3 pad 8: L_K15 -> /left/C4
- J3 pad 9: L_K6 -> /left/C3
- J3 pad MP: (no net) -> /left/GND
- J4 pad 10: K10 -> C2
- J4 pad 11: K9 -> C1
- J4 pad 12: K8 -> C0
- J4 pad 2: BAT -> GND
- J4 pad 3: GND -> unconnected-(J4-Pad3)
- J4 pad 4: GND -> R3
- J4 pad 5: K5 -> R2
- J4 pad 6: K4 -> R1
- J4 pad 7: K3 -> R0
- J4 pad 8: K2 -> C4
- J4 pad 9: K1 -> C3
- J4 pad MP: (no net) -> GND
- JP1 pad 1: MAGNET -> VDD
- JP1 pad 2: Net-(JP1-Pad2) -> +2V8
- K1 pad 1: L_K1 -> /left/R0
- K1 pad 2: L_GND -> /left/C0
- K10 pad 1: L_K10 -> /left/R1
- K10 pad 2: L_GND -> /left/C4
- K11 pad 1: L_K11 -> /left/R2
- K11 pad 2: L_GND -> /left/C0
- K12 pad 1: L_K12 -> /left/R2
- K12 pad 2: L_GND -> /left/C1
- K13 pad 1: L_K13 -> /left/R2
- K13 pad 2: L_GND -> /left/C2
- K14 pad 1: L_K14 -> /left/R2
- K14 pad 2: L_GND -> /left/C3
- K15 pad 1: L_K15 -> /left/R2
- K15 pad 2: L_GND -> /left/C4
- K16 pad 1: L_K16 -> /left/R3
- K16 pad 2: L_GND -> /left/C2
- K17 pad 1: L_K17 -> /left/R3
- K17 pad 2: L_GND -> /left/C3
- K18 pad 1: L_K18 -> /left/R3
- K18 pad 2: L_GND -> /left/C4
- K19 pad 1: K19 -> R4
- K19 pad 2: GND -> C0
- K2 pad 1: L_K2 -> /left/R0
- K2 pad 2: L_GND -> /left/C1
- K20 pad 1: K20 -> R4
- K20 pad 2: GND -> C1
- K21 pad 1: K21 -> R4
- K21 pad 2: GND -> C2
- K22 pad 1: K22 -> R4
- K22 pad 2: GND -> C3
- K23 pad 1: K23 -> R4
- K23 pad 2: GND -> C4
- K24 pad 1: K24 -> R5
- K24 pad 2: GND -> C0
- K25 pad 1: K25 -> R5
- K25 pad 2: GND -> C1
- K26 pad 1: K26 -> R5
- K26 pad 2: GND -> C2
- K27 pad 1: K27 -> R5
- K27 pad 2: GND -> C3
- K28 pad 1: K28 -> R5
- K28 pad 2: GND -> C4
- K29 pad 1: K29 -> R6
- K29 pad 2: GND -> C0
- K3 pad 1: L_K3 -> /left/R0
- K3 pad 2: L_GND -> /left/C2
- K30 pad 1: K30 -> R6
- K30 pad 2: GND -> C1
- K31 pad 1: K31 -> R6
- K31 pad 2: GND -> C2
- K32 pad 1: K32 -> R6
- K32 pad 2: GND -> C3
- K33 pad 1: K33 -> R6
- K33 pad 2: GND -> C4
- K34 pad 1: K34 -> R7
- K34 pad 2: GND -> C0
- K35 pad 1: K35 -> R7
- K35 pad 2: GND -> C1
- K36 pad 1: K36 -> R7
- K36 pad 2: GND -> C2
- K37 pad 1: K37 -> R7
- K37 pad 2: GND -> C3
- K38 pad 1: K38 -> R7
- K38 pad 2: GND -> C4
- K4 pad 1: L_K4 -> /left/R0
- K4 pad 2: L_GND -> /left/C3
- K5 pad 1: L_K5 -> /left/R0
- K5 pad 2: L_GND -> /left/C4
- K6 pad 1: L_K6 -> /left/R1
- K6 pad 2: L_GND -> /left/C0
- K7 pad 1: L_K7 -> /left/R1
- K7 pad 2: L_GND -> /left/C1
- K8 pad 1: L_K8 -> /left/R1
- K8 pad 2: L_GND -> /left/C2
- K9 pad 1: L_K9 -> /left/R1
- K9 pad 2: L_GND -> /left/C3
- R10 pad 2: MAGNET -> Net-(JP6-Pad1)
- U1 pad 10: K30 -> TRACKPAD_~{CS}
- U1 pad 11: K29 -> MOTION
- U1 pad 12: K37 -> SHTDWN
- U1 pad 14: K25 -> unconnected-(U1-Pad14)
- U1 pad 15: K26 -> unconnected-(U1-Pad15)
- U1 pad 16: K27 -> unconnected-(U1-Pad16)
- U1 pad 17: K23 -> unconnected-(U1-Pad17)
- U1 pad 2: K34 -> unconnected-(U1-Pad2)
- U1 pad 23: K4 -> unconnected-(U1-Pad23)
- U1 pad 24: K2 -> unconnected-(U1-Pad24)
- U1 pad 25: K10 -> unconnected-(U1-Pad25)
- U1 pad 26: K8 -> unconnected-(U1-Pad26)
- U1 pad 27: K6 -> unconnected-(U1-Pad27)
- U1 pad 28: K14 -> unconnected-(U1-Pad28)
- U1 pad 29: K12 -> unconnected-(U1-Pad29)
- U1 pad 3: K35 -> unconnected-(U1-Pad3)
- U1 pad 30: K16 -> unconnected-(U1-Pad30)
- U1 pad 31: K17 -> unconnected-(U1-Pad31)
- U1 pad 33: K5 -> R3
- U1 pad 34: K3 -> R2
- U1 pad 35: K1 -> R1
- U1 pad 36: K9 -> R0
- U1 pad 39: K7 -> unconnected-(U1-Pad39)
- U1 pad 4: K36 -> unconnected-(U1-Pad4)
- U1 pad 40: K15 -> unconnected-(U1-Pad40)
- U1 pad 41: K13 -> unconnected-(U1-Pad41)
- U1 pad 42: K11 -> unconnected-(U1-Pad42)
- U1 pad 43: K18 -> unconnected-(U1-Pad43)
- U1 pad 5: K33 -> unconnected-(U1-Pad5)
- U1 pad 50: K19 -> R4
- U1 pad 51: K20 -> R5
- U1 pad 52: K21 -> R6
- U1 pad 53: K22 -> R7
- U1 pad 54: K24 -> unconnected-(U1-Pad54)
- U1 pad 6: K38 -> unconnected-(U1-Pad6)
- U1 pad 7: K28 -> unconnected-(U1-Pad7)
- U1 pad 8: K32 -> unconnected-(U1-Pad8)
- U1 pad 9: K31 -> unconnected-(U1-Pad9)
- U4 pad 3: Net-(JP1-Pad2) -> Net-(JP6-Pad2)
- U5 pad 2: MAGNET -> Net-(JP6-Pad1)
Routing:
- net L_GND: track 361.2 -> 0.00 mm
- net GND: track 481.9 -> 176.4 mm, vias 17 -> 24
- net R7: track 0.00 -> 195.5 mm, vias 0 -> 1
- net C4: track 0.00 -> 174.4 mm, vias 0 -> 4
- net C2: track 0.00 -> 154.0 mm, vias 0 -> 2
- net /left/C0: track 0.00 -> 150.8 mm
- net C3: track 0.00 -> 150.7 mm, vias 0 -> 2
- net /left/R2: track 0.00 -> 134.8 mm, vias 0 -> 1
- net /left/C2: track 0.00 -> 133.4 mm
- net L_K6: track 132.6 -> 0.00 mm
- net L_K11: track 130.6 -> 0.00 mm
- net R4: track 0.00 -> 128.8 mm, vias 0 -> 1
- net C1: track 0.00 -> 127.2 mm, vias 0 -> 2
- net /left/R1: track 0.00 -> 126.5 mm, vias 0 -> 1
- net R6: track 0.00 -> 124.6 mm, vias 0 -> 1
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Other:
- board size 276.3 x 95.6 mm -> 406.7 x 118.7 mm

Commit message: trackpad
Parts:
- removed J6: trackpad_conn, fusion:trackpad_conn
- removed J7: Conn_02x10_Odd_Even_MountingPin, keeb-libs:hirose-df30fb-20ds-0.4v(82)
- removed the REF** at (157.5, 121.9)
- removed the REF** at (157.5, 166.5)
- removed the REF** at (69.7, 94.3)
- removed the REF** at (26.1, 98.7)
- removed the REF** at (26.1, 143.3)
- added H1: trackpad, fusion:trackpad, F.Cu at (126.9, 195.3)
- added H10: hinge, fusion:hinge, F.Cu at (96.9, 182.8)
- added H11: hinge-big, fusion:hinge-big, F.Cu at (119.6, 94.8)
- added H12: hinge-big, fusion:hinge-big, F.Cu at (106.6, 139.4)
- added H13: hinge-small, fusion:hinge-small, F.Cu at (106.6, 94.8)
- added H14: hinge-small, fusion:hinge-small, F.Cu at (119.6, 139.4)
- added H2: trackpad, fusion:trackpad, F.Cu at (126.9, 177.3)
- added H3: trackpad, fusion:trackpad, B.Cu at (191.6, 153.2)
- added H4: trackpad, fusion:trackpad, B.Cu at (187.0, 135.8)
- added H5: hinge, fusion:hinge, B.Cu at (102.9, 182.8)
- added H6: hinge, fusion:hinge, B.Cu at (96.9, 182.8)
- added H7: hinge, fusion:hinge, F.Cu at (91.4, 182.8)
- added H8: hinge, fusion:hinge, B.Cu at (91.4, 182.8)
- added H9: hinge, fusion:hinge, F.Cu at (102.9, 182.8)
- added REF**: magnet-fp, fusion:magnet-fp, B.Cu at (228.9, 83.4)
- J5: value trackpad -> Conn_02x10_Odd_Even_MountingPin; footprint fusion:trackpad -> keeb-libs:hirose-df30fb-20ds-0.4v(82)
- moved R11 140.3 mm to (215.1, 130.9), turned to 15 degrees
- moved R4 138.9 mm to (212.2, 131.6), turned to 15 degrees
- moved C6 132.6 mm to (214.1, 132.7), turned to 15 degrees
- moved J5 122.7 mm to (212.2, 127.6), turned to 15 degrees
- moved BT1 80.7 mm to (80.9, 87.8)
- moved J3 80.7 mm to (91.6, 103.3)
- moved K1 80.7 mm to (-2.02, 95.9)
- moved K10 80.7 mm to (65.8, 107.4)
- moved K15 80.7 mm to (62.3, 120.4)
- moved K5 80.7 mm to (69.3, 94.3)
- moved REF** 80.7 mm to (-3.58, 83.0)
- moved K11 80.7 mm to (-6.78, 122.6)
- moved K12 80.7 mm to (13.6, 107.3)
- moved K13 80.7 mm to (32.8, 105.2)
- moved K14 80.7 mm to (48.3, 116.7)
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Connections:
- C6 pad 1: /trackpad/2V8 -> +2V8
- C6 pad 2: /trackpad/GND -> GND
- J5 pad 1: /trackpad/2V8 -> GND
- J5 pad 2: /trackpad/GND -> unconnected-(J5-Pad2)
- J5 pad 3: /trackpad/MOTION_2V8 -> unconnected-(J5-Pad3)
- J5 pad 4: /trackpad/MISO_2V8 -> unconnected-(J5-Pad4)
- J5 pad 5: /trackpad/MOSI_2V8 -> GND
- J5 pad 6: /trackpad/SCK_2V8 -> unconnected-(J5-Pad6)
- J5 pad 7: /trackpad/~{CS}_2V8 -> SHTDWN_2V8
- J5 pad 8: /trackpad/SHTDWN_2V8 -> unconnected-(J5-Pad8)
- JP2 pad 2: /trackpad_conn/SHTDWN_2V8 -> SHTDWN_2V8
- JP3 pad 2: /trackpad_conn/~{CS}_2V8 -> ~{CS}_2V8
- JP4 pad 2: /trackpad_conn/SCK_2V8 -> SCK_2V8
- JP5 pad 2: /trackpad_conn/MOSI_2V8 -> MOSI_2V8
- R11 pad 1: Net-(J7-Pad14) -> /trackpad_conn/R11_conn
- R11 pad 2: /trackpad/GND -> GND
- R4 pad 1: Net-(J7-Pad10) -> /trackpad_conn/R4_conn
- R4 pad 2: /trackpad/2V8 -> +2V8
- U1 pad 10: TRACKPAD_~{CS} -> SHTDWN
- U1 pad 11: MOTION -> TRACKPAD_~{CS}
- U1 pad 12: SHTDWN -> MOTION
- U7 pad 10: /trackpad_conn/MOSI_2V8 -> MOSI_2V8
- U7 pad 2: /trackpad_conn/SHTDWN_2V8 -> SHTDWN_2V8
- U7 pad 4: /trackpad_conn/~{CS}_2V8 -> ~{CS}_2V8
- U7 pad 6: /trackpad_conn/SCK_2V8 -> SCK_2V8
Routing:
- net Net-(JP6-Pad1): track 93.5 -> 10.1 mm, vias 2 -> 0
- net VDDH: track 124.5 -> 57.7 mm
- net GND: track 176.4 -> 126.0 mm, vias 24 -> 19
- net MOSI_DQ0: track 119.0 -> 83.8 mm
- net /trackpad/GND: track 31.5 -> 0.00 mm, vias 2 -> 0
- net /trackpad_conn/MOSI_2V8: track 24.3 -> 0.00 mm
- net /trackpad/2V8: track 24.0 -> 0.00 mm
- net MOSI_2V8: track 0.00 -> 22.9 mm
- net SHTDWN_2V8: track 0.00 -> 18.0 mm
- net ~{CS}_2V8: track 0.00 -> 15.3 mm
- net SCLK: track 106.7 -> 91.8 mm
- net SCK_2V8: track 0.00 -> 14.5 mm
- net MISO_DQ1: track 78.4 -> 92.6 mm, vias 2 -> 3
- net /trackpad/MOTION_2V8: track 13.4 -> 0.00 mm
- net /trackpad_conn/SCK_2V8: track 12.5 -> 0.00 mm
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Other:
- board size 406.7 x 118.7 mm -> 288.3 x 122.1 mm
- board text added: "mag"
- board text added: "rough shadow of a 45 deg trackpad"

Commit message: use narrower pinky spacing
Parts:
- K1, K11, K37, K38, K6: footprint pg1232:pg1232-DSSR -> pg1232:pg1232-DSSN
- K12, K2, K7: footprint pg1232:pg1232-DSS -> pg1232:pg1232-DSSR
- K22, K27, K32: footprint pg1232:pg1232-DSS -> pg1232:pg1232-DSSL
- K23, K28, K33: footprint pg1232:pg1232-DSSL -> pg1232:pg1232-DSSN
- moved H3 8.57 mm to (198.5, 148.1)
- moved J2 8.57 mm to (151.1, 73.4)
- moved K26 8.57 mm to (196.9, 87.1)
- moved D1 8.57 mm to (159.4, 72.7)
- moved JP4 8.57 mm to (210.5, 122.5)
- moved K20 8.57 mm to (177.8, 85.5)
- moved K27 8.57 mm to (216.1, 89.2)
- moved K29 8.57 mm to (170.8, 115.3)
- moved K31 8.57 mm to (200.4, 100.1)
- moved R1 8.57 mm to (139.9, 78.7)
- moved R7 8.57 mm to (153.5, 80.0)
- moved U1 8.57 mm to (137.8, 115.5)
- moved U4 8.57 mm to (148.4, 83.9)
- moved H14 8.57 mm to (126.5, 134.3)
- moved C3 8.57 mm to (145.5, 81.6)
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Routing:
- net /left/C0: track 150.5 -> 145.6 mm
- net C3: track 154.0 -> 150.7 mm
- net C4: track 179.9 -> 176.9 mm
- net R4: track 128.8 -> 126.0 mm
- net R7: track 192.1 -> 194.5 mm
- net /left/R1: track 126.5 -> 125.8 mm
- net /left/R0: track 114.1 -> 113.5 mm
Other:
- board size 288.3 x 122.1 mm -> 285.6 x 127.3 mm

Commit message: final?
Parts:
- removed D42: SK6812MINI, LED_SMD:LED_SK6812MINI_PLCC4_3.5x3.5mm_P1.75mm
- removed JP1, JP2, JP3, JP4, JP5: SolderJumper_2_Open, Jumper:SolderJumper-2_P1.3mm_Open_RoundedPad1.0x1.5mm
- removed JP6: Jumper_3_Open, Jumper:SolderJumper-3_P2.0mm_Open_TrianglePad1.0x1.5mm_NumberLabels
- removed REF** (x2): magnet-fp, fusion:magnet-fp
- added D2: LED_RBAG, fusion:FM-B2020RGBA, F.Cu at (156.9, 102.1)
- added H15: sensor-magnet, fusion:sensor-magnet, F.Cu at (43.1, 111.8)
- added H16: mount-magnet, fusion:mount-magnet, F.Cu at (227.1, 73.8)
- added H17: mount-magnet, fusion:mount-magnet, F.Cu at (244.6, 79.1)
- added H18: mount-magnet, fusion:mount-magnet, F.Cu at (253.1, 114.8)
- added H19: mount-magnet, fusion:mount-magnet, F.Cu at (231.4, 128.1)
- added R12: 1.2k, Resistor_SMD:R_0603_1608Metric, F.Cu at (158.4, 105.6)
- added R13: 1.5k, Resistor_SMD:R_0603_1608Metric, F.Cu at (156.9, 105.6)
- added R14: 1k, Resistor_SMD:R_0603_1608Metric, F.Cu at (155.4, 105.6)
- added SW2: SW_SPDT, Button_Switch_SMD:SW_SPDT_PCM12, F.Cu at (164.4, 69.6)
- H10, H7, H9: value hinge -> mount-magnet; footprint fusion:hinge -> fusion:mount-magnet
- H6: moved to F.Cu
- H8: value hinge -> mount-magnet; footprint fusion:hinge -> fusion:mount-magnet; moved to F.Cu
- J1: footprint keeb-libs:debug-port -> keeb-libs:debug-port-single-side
- R3: value 10k -> 100k
- U1: value Holyiot_18010 -> Holyiot_18010_no_underside; footprint keeb-libs:Holyiot-18010 -> keeb-libs:Holyiot-18010-no-underside
- U6: footprint Package_TO_SOT_SMD:SOT-353_SC-70-5 -> Package_TO_SOT_SMD:SOT-23-5
- moved H1 143.5 mm to (152.1, 54.0)
- moved H2 143.5 mm to (152.1, 36.0)
- moved H6 139.9 mm to (137.2, 48.8)
- moved H5 138.3 mm to (137.2, 48.8)
- moved H8 135.3 mm to (4.39, 79.1)
- moved H7 129.2 mm to (21.9, 73.8)
- moved H9 126.7 mm to (-4.11, 114.8)
- moved H10 96.3 mm to (17.6, 128.1)
- moved C5 46.3 mm to (205.3, 109.4), turned to 15 degrees
- moved R10 46.3 mm to (203.5, 112.5), turned to -75 degrees
- moved U5 45.9 mm to (205.9, 111.8), turned to 15 degrees
- moved J1 34.1 mm to (135.5, 75.7), turned to 180 degrees
- moved SW1 26.0 mm to (156.9, 98.3), turned to 0 degrees
- moved C6 19.8 mm to (201.2, 129.1), turned to -165 degrees
- moved J3 15.2 mm to (106.4, 95.1)
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Connections:
- net /trackpad_conn/R11_conn renamed Net-(J5-Pad14)
- net /trackpad_conn/R4_conn renamed Net-(J5-Pad10)
- J1 pad 3: SWD -> SWC
- J1 pad 4: SWC -> SWD
- J5 pad 16: unconnected-(J5-Pad16) -> /trackpad-8520/KEY_OUT
- J5 pad 18: unconnected-(J5-Pad18) -> /trackpad-8520/KEY_IN
- R10 pad 2: Net-(JP6-Pad1) -> MAGNET
- U1 pad 10: SHTDWN -> TRACKPAD_~{CS}
- U1 pad 11: TRACKPAD_~{CS} -> BAT_MEAS
- U1 pad 12: MOTION -> MISO_DQ1
- U1 pad 13: BAT_MEAS -> MOSI_DQ0
- U1 pad 2: unconnected-(U1-Pad2) -> R3
- U1 pad 3: unconnected-(U1-Pad3) -> R2
- U1 pad 33: R3 -> C4
- U1 pad 34: R2 -> C3
- U1 pad 35: R1 -> C2
- U1 pad 36: R0 -> C1
- U1 pad 39: unconnected-(U1-Pad39) -> C0
- U1 pad 4: unconnected-(U1-Pad4) -> R1
- U1 pad 40: unconnected-(U1-Pad40) -> MAGNET
- U1 pad 41: unconnected-(U1-Pad41) -> R4
- U1 pad 43: unconnected-(U1-Pad43) -> R5
- U1 pad 49: RGB -> ~{BLUE}
- U1 pad 5: unconnected-(U1-Pad5) -> R0
- U1 pad 50: R4 -> ~{GREEN}
- U1 pad 51: R5 -> ~{RED}
- U1 pad 54: unconnected-(U1-Pad54) -> SCLK
- U1 pad 6: unconnected-(U1-Pad6) -> DISP_~{CS}
- U1 pad 7: unconnected-(U1-Pad7) -> MOTION
- U1 pad 8: unconnected-(U1-Pad8) -> FLASH_~{CS}
- U1 pad 9: unconnected-(U1-Pad9) -> SHTDWN
- U5 pad 2: Net-(JP6-Pad1) -> MAGNET
- U7 pad 10: MOSI_2V8 -> (no net)
- U7 pad 11: (no net) -> MOSI_DQ0
- U7 pad 12: (no net) -> MOSI_2V8
- U7 pad 14: (no net) -> TRACKPAD_~{CS}
- U7 pad 15: (no net) -> ~{CS}_2V8
- U7 pad 4: ~{CS}_2V8 -> SCK_2V8
- U7 pad 5: TRACKPAD_~{CS} -> SCLK
- U7 pad 6: SCK_2V8 -> (no net)
- U7 pad 7: SCLK -> (no net)
- U7 pad 9: MOSI_DQ0 -> (no net)
Routing:
- net MAGNET: track 0.00 -> 109.8 mm, vias 0 -> 3
- net GND: track 126.0 -> 46.7 mm, vias 19 -> 29
- net VDDH: track 57.7 -> 101.3 mm, vias 4 -> 3
- net RST: track 45.8 -> 15.2 mm
- net SWC: track 60.6 -> 33.4 mm
- net SWD: track 60.0 -> 35.3 mm
- net RGB: track 23.2 -> 0.00 mm
- net VDD: track 165.0 -> 148.7 mm, vias 8 -> 7
- net R3: track 18.6 -> 34.1 mm, vias 0 -> 2
- net C2: track 161.3 -> 176.7 mm
- net R2: track 17.4 -> 32.6 mm, vias 0 -> 2
- net R1: track 16.1 -> 31.2 mm, vias 0 -> 2
- net R0: track 14.9 -> 29.7 mm, vias 0 -> 2
- net C3: track 150.7 -> 164.8 mm
- net MISO_DQ1: track 92.6 -> 79.0 mm, vias 3 -> 2
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Other:
- board size 285.6 x 127.3 mm -> 272.9 x 124.2 mm
- board text added: "DC"
