File: fusion.kicad_pcb (KiCad board)
At the start: 2 copper layers, 272.9 x 124.2 mm, 95 parts, among them J1 Conn_01x04_Female, J2 USB_C_Receptacle_USB2.0, J3 Conn_01x12_MountingPin, J4 Conn_01x12_MountingPin, J5 Conn_02x10_Odd_Even_MountingP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, K1 diode-choc, K10 diode-choc, K11 diode-choc, K12 diode-choc, K13 diode-choc, K14 diode-choc, K15 diode-choc, K16 diode-choc, K17 diode-choc, K18 diode-choc, K19 diode-choc, K2 diode-choc, K20 diode-choc, K21 diode-choc, K22 diode-choc, K23 diode-choc, K24 diode-choc, K25 diode-choc, K26 diode-choc, K27 diode-choc, K28 diode-choc, K29 diode-choc, K3 diode-choc, K30 diode-choc, K31 diode-choc, K32 diode-choc, K33 diode-choc, K34 diode-choc, K35 diode-choc, K36 diode-choc, K37 diode-choc, K38 diode-choc, K4 diode-choc, K5 diode-choc, K6 diode-choc, K7 diode-choc, K8 diode-choc, K9 diode-choc, SW1 SW_Push, SW2 SW_SPDT, U1 Holyiot_18010_no_underside, U2 MT25QL128ABA1ESE, U3 BQ24075, U4 XC6220B331MR, U5 LN4913, U6 MIC5365-2.8YC5, U7 4050

Commit message: backup
Parts:
- removed H10, H16, H19: mount-magnet, fusion:mount-magnet
- added H20: bat-cover, fusion:bat-cover, F.Cu at (96.6, 139.5)
- added H21: hinge-mousebite, fusion:hinge-mousebite, F.Cu at (130.9, 44.2)
- added H22: hinge-mousebite, fusion:hinge-mousebite, F.Cu at (134.6, 44.3)
- added H23: hinge-mousebite, fusion:hinge-mousebite, F.Cu at (143.8, 44.2)
- added H24: hinge-mousebite, fusion:hinge-mousebite, F.Cu at (140.2, 44.2)
- added JP1: SolderJumper_2_Open, Jumper:SolderJumper-2_P1.3mm_Open_RoundedPad1.0x1.5mm, F.Cu at (183.7, 129.4)
- added JP2: SolderJumper_2_Open, Jumper:SolderJumper-2_P1.3mm_Open_RoundedPad1.0x1.5mm, F.Cu at (174.3, 132.5)
- added JP3: SolderJumper_2_Open, Jumper:SolderJumper-2_P1.3mm_Open_RoundedPad1.0x1.5mm, F.Cu at (179.0, 132.1)
- added REF**: hinge1, fusion:hinge1, F.Cu at (160.4, 131.5)
- added REF**: hinge2, fusion:hinge2, F.Cu at (160.4, 89.5)
- added REF**: hinge2, fusion:hinge2, F.Cu at (138.8, 131.5)
- added REF**: hinge1, fusion:hinge1, F.Cu at (138.8, 89.5)
- added U8: SRV05-4, Package_TO_SOT_SMD:SOT-23-6, F.Cu at (184.6, 89.7)
- D2: value LED_RBAG -> LED_RABG; footprint fusion:FM-B2020RGBA -> LED_SMD:LED_ASMB-KTF0-0A306
- H5: moved to F.Cu
- H7: value mount-magnet -> hinge; footprint fusion:mount-magnet -> fusion:hinge
- K19, K24, K29: footprint pg1232:pg1232-DSSL -> pg1232:pg1232-DSSN
- K20, K25, K30: footprint pg1232:pg1232-DSSR -> pg1232:pg1232-DSSL
- K22, K27, K32: footprint pg1232:pg1232-DSSL -> pg1232:pg1232-DSSR
- K23, K28, K33: footprint pg1232:pg1232-DSSN -> pg1232:pg1232-DSSL
- K34, K35: footprint pg1232:pg1232-DSS -> pg1232:pg1232-DSSN
- K37, K38: footprint pg1232:pg1232-DSSN -> pg1232:pg1232-DSS
- moved K34 121.5 mm to (283.4, 99.1), turned to 15 degrees
- moved K35 110.5 mm to (279.9, 86.1), turned to 15 degrees
- moved H7 108.2 mm to (127.4, 49.9)
- moved K29 100.5 mm to (272.9, 115.9)
- moved K24 100.5 mm to (269.4, 102.9)
- moved K19 100.5 mm to (265.9, 89.9)
- moved K38 67.8 mm to (204.1, 147.7), turned to -75 degrees
- moved K20 67.6 mm to (246.5, 73.3)
- moved K25 67.6 mm to (250.0, 86.4)
- moved K30 67.6 mm to (253.5, 99.4)
- moved K37 64.1 mm to (216.5, 141.8), turned to -75 degrees
- moved H9 43.6 mm to (39.5, 114.7)
- moved K28 36.1 mm to (201.2, 99.4)
- moved K33 36.1 mm to (204.7, 112.5)
- moved K23 36.1 mm to (197.7, 86.4)
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Connections:
- D2 pad 2: Net-(D2-Pad2) -> VDD
- D2 pad 3: VDD -> Net-(D2-Pad3)
- J3 pad 1: /left/BAT -> /left/R3
- J3 pad 10: /left/C2 -> unconnected-(J3-Pad10)
- J3 pad 11: /left/C1 -> /left/GND
- J3 pad 12: /left/C0 -> /left/BAT
- J3 pad 2: /left/GND -> /left/R2
- J3 pad 3: unconnected-(J3-Pad3) -> /left/R1
- J3 pad 4: /left/R3 -> /left/R0
- J3 pad 5: /left/R2 -> /left/C4
- J3 pad 6: /left/R1 -> /left/C3
- J3 pad 7: /left/R0 -> /left/C2
- J3 pad 8: /left/C4 -> /left/C1
- J3 pad 9: /left/C3 -> /left/C0
- J4 pad 10: C2 -> R1
- J4 pad 11: C1 -> R2
- J4 pad 12: C0 -> R3
- J4 pad 4: R3 -> C0
- J4 pad 5: R2 -> C1
- J4 pad 6: R1 -> C2
- J4 pad 7: R0 -> C3
- J4 pad 9: C3 -> R0
- J5 pad 15: MISO_DQ1 -> /trackpad-8520/MISO_2V8
- R14 pad 2: Net-(D2-Pad2) -> Net-(D2-Pad3)
- U1 pad 2: R3 -> C0
- U1 pad 3: R2 -> C1
- U1 pad 34: C3 -> R0
- U1 pad 35: C2 -> R1
- U1 pad 36: C1 -> R2
- U1 pad 39: C0 -> R3
- U1 pad 4: R1 -> C2
- U1 pad 5: R0 -> C3
- U1 pad 53: R7 -> FLASH_~{CS}
- U1 pad 8: FLASH_~{CS} -> R7
- U7 pad 11: MOSI_DQ0 -> /trackpad-8520/MOSI_3V3
- U7 pad 5: SCLK -> /trackpad-8520/SCK_3V3
Routing:
- net C0: track 122.1 -> 200.2 mm, vias 2 -> 6
- net /trackpad-8520/MISO_2V8: track 0.00 -> 67.6 mm, vias 0 -> 2
- net /trackpad-8520/MOSI_3V3: track 0.00 -> 65.9 mm, vias 0 -> 2
- net MISO_DQ1: track 79.0 -> 15.1 mm, vias 2 -> 0
- net MOSI_DQ0: track 81.5 -> 19.1 mm, vias 2 -> 0
- net SCLK: track 81.7 -> 24.6 mm, vias 2 -> 0
- net /trackpad-8520/SCK_3V3: track 0.00 -> 56.0 mm, vias 0 -> 2
- net C4: track 179.5 -> 128.1 mm, vias 4 -> 2
- net C1: track 141.1 -> 177.8 mm, vias 2 -> 4
- net R3: track 34.1 -> 7.28 mm, vias 2 -> 0
- net R2: track 32.6 -> 11.3 mm, vias 2 -> 0
- net R1: track 31.2 -> 12.5 mm, vias 2 -> 0
- net C2: track 176.7 -> 192.9 mm, vias 2 -> 4
- net R0: track 29.7 -> 13.8 mm, vias 2 -> 0
- net Net-(D2-Pad3): track 0.00 -> 12.7 mm
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Other:
- board size 272.9 x 124.2 mm -> 287.3 x 124.3 mm
- board text added: "MISO"
- board text added: "MOSI"
- board text added: "SCLK"

Commit message: Hydrogen.PCB
- add Adafruit CAD files for Sharp display
- convert to all 3D printed mechanical parts
- update part dimensions to lowest estimate
Parts:
- removed the H2 at (161.5, 36.2)
- removed H21, H22, H23, H24: hinge-mousebite, fusion:hinge-mousebite
- removed H3: trackpad, fusion:trackpad
- removed the H4 at (227.7, 127.9)
- removed H5, H6, H7: hinge, fusion:hinge
- removed REF** (x2): hinge1, fusion:hinge1
- removed REF** (x2): hinge2, fusion:hinge2
- added H2: mouse-bite, Keebio-Parts:breakaway-mousebites, F.Cu at (159.0, 48.2)
- added H2: mouse-bite, Keebio-Parts:breakaway-mousebites, B.Cu at (39.5, 48.2)
- added H4: mouse-bite, Keebio-Parts:breakaway-mousebites, F.Cu at (127.8, 54.2)
- added H4: mouse-bite, Keebio-Parts:breakaway-mousebites, B.Cu at (70.7, 54.2)
- BT1: footprint Connector_JST:JST_PH_S2B-PH-K_1x02_P2.00mm_Horizontal -> Connector_JST:JST_PH_S2B-PH-SM4-TB_1x02-1MP_P2.00mm_Horizontal
- H1: value trackpad -> touchpad; footprint fusion:trackpad -> fusion:touchpad-holder
- H11, H12: footprint fusion:hinge-big -> fusion:hinge2
- H13, H14: footprint fusion:hinge-small -> fusion:hinge1
- H20: value bat-cover -> bat-shell; footprint fusion:bat-cover -> fusion:bat-shell
- SW1: footprint Button_Switch_SMD:SW_SPST_B3U-1000P -> Button_Switch_SMD:SW_SPST_TL3342
- moved H1 61.9 mm to (185.1, 111.4), turned to 15 degrees
- moved C1 61.4 mm to (123.6, 74.1), turned to 180 degrees
- moved C6 60.6 mm to (177.2, 107.0)
- moved H17 60.4 mm to (206.0, 60.7)
- moved U6 60.3 mm to (177.7, 109.6)
- moved H11 60.3 mm to (104.5, 66.9)
- moved H18 60.3 mm to (203.5, 92.8)
- moved SW1 60.3 mm to (133.2, 77.5), turned to 90 degrees
- moved D2 60.2 mm to (132.5, 71.5)
- moved H14 60.1 mm to (104.5, 109.3)
- moved R1 60.1 mm to (119.5, 68.4)
- moved R3 60.1 mm to (126.1, 100.9)
- moved K27 60.1 mm to (159.3, 73.5)
- moved C3 60.1 mm to (120.2, 61.3)
- moved K33 60.1 mm to (148.8, 90.3)
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Connections:
- J5 pad 16: /trackpad-8520/KEY_OUT -> GND
- J5 pad 18: /trackpad-8520/KEY_IN -> TOUCHPAD_BTN
- U1 pad 42: unconnected-(U1-Pad42) -> R5
- U1 pad 43: R5 -> TOUCHPAD_BTN
- U1 pad 6: DISP_~{CS} -> R7
- U1 pad 7: MOTION -> DISP_~{CS}
- U1 pad 8: R7 -> MOTION
Routing:
- net TOUCHPAD_BTN: track 0.00 -> 80.6 mm, vias 0 -> 2
- net GND: track 53.2 -> 71.7 mm, vias 30 -> 29
- net RST: track 16.3 -> 19.7 mm
- net SWD: track 31.5 -> 28.9 mm
- net /trackpad-8520/MISO_2V8: track 67.6 -> 69.9 mm
- net Net-(J5-Pad10): track 2.88 -> 5.04 mm
- net SWC: track 30.1 -> 28.1 mm
- net /left/C0: track 152.8 -> 154.6 mm
- net VDD: track 141.1 -> 139.4 mm
- net C0: track 200.2 -> 198.5 mm
- net /left/C3: track 112.0 -> 113.5 mm
- net R5: track 124.9 -> 126.4 mm
- net /left/C2: track 135.6 -> 137.1 mm
- net BAT: track 14.2 -> 15.7 mm
- net R0: track 13.8 -> 12.3 mm
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Other:
- board size 287.3 x 124.3 mm -> 276.2 x 92.3 mm
- board text added: "JLCJLCJLCJLC"
