File: fusion.kicad_pcb (KiCad board)
At the start: 2 copper layers, 280 x 97 mm, 130 parts, among them J1 tc2030, J2 USB_C_Receptacle_USB2.0, J3 Conn_01x12_MountingPin, J4 Conn_01x12_MountingPin, J5 cirque-trackpad, K1 diode-choc, K10 diode-choc, K11 diode-choc, K12 diode-choc, K13 diode-choc, K14 diode-choc, K15 diode-choc, K16 diode-choc, K17 diode-choc, K18 diode-choc, K19 diode-choc, K2 diode-choc, K20 diode-choc, K21 diode-choc, K22 diode-choc, K23 diode-choc, K24 diode-choc, K25 diode-choc, K26 diode-choc, K27 diode-choc, K28 diode-choc, K29 diode-choc, K3 diode-choc, K30 diode-choc, K31 diode-choc, K32 diode-choc, K33 diode-choc, K34 diode-choc, K35 diode-choc, K36 diode-choc, K37 diode-choc, K38 diode-choc, K4 diode-choc, K5 diode-choc, K6 diode-choc, K7 diode-choc, K8 diode-choc, K9 diode-choc, SW1 SW_Push, SW2 SW_SPDT, U1 holyiot-18010-no-underside, U2 MT25QL128ABA1ESE, U3 BQ24075, U4 XC6206B331MR, U5 LN4913, U8 SRV05-4

Commit message: backup & remove useless things
Parts:
- removed BT1: Battery_Cell, Connector_JST:JST_PH_S2B-PH-SM4-TB_1x02-1MP_P2.00mm_Horizontal
- removed H20: bat-shell, fusion:bat-shell-small
- removed K34, K35: diode-choc, pg1232:pg1232-DSSN
- removed the REF** at (225.5, 61.7)
- removed the REF** at (75.8, 61.7)
- removed the REF** at (108.3, 68.2) (x2)
- removed the REF** at (70.6, 74.2)
- removed the REF** at (103.2, 80.7)
- removed the REF** at (71.0, 113.5)
- removed the REF** at (94.9, 62.6)
- removed the REF** at (279.7, 69.6)
- removed the REF** at (274.5, 57.2)
- removed the REF** at (40.2, 62.7)
- removed the REF** at (239.7, 48.9)
- removed the REF** at (220.4, 49.3)
- removed the REF** at (82.6, 120.5)
- removed the REF** at (98.0, 93.1)
- removed the REF** at (89.8, 75.1)
- removed the REF** at (211.6, 75.1)
- removed the REF** at (271.4, 87.7)
- removed the REF** at (51.3, 73.8)
- removed the REF** at (193.0, 68.2)
- removed the REF** at (230.4, 113.6)
- removed the REF** at (230.7, 74.2)
- removed the REF** at (61.7, 48.9)
- removed the REF** at (203.4, 93.1)
- removed the REF** at (29.9, 87.7)
- removed the REF** at (35.1, 75.2)
- removed the REF** at (81.0, 49.3)
- removed the REF** at (206.4, 62.6)
- removed the REF** at (56.5, 61.3)
- removed the REF** at (244.8, 61.3)
- removed the REF** at (250.0, 73.8)
- removed the REF** at (84.6, 87.6)
- removed the REF** at (261.1, 62.7)
- removed the REF** at (218.8, 120.5)
- removed the REF** at (207.2, 127.4)
- removed the REF** at (94.1, 127.4)
- removed the REF** at (216.7, 87.6)
- removed the REF** at (198.2, 80.7)
- removed the REF** at (266.3, 75.2)
- removed the U4 at (176.2, 81.7)
- added C6: 0.1uF, Capacitor_SMD:C_0603_1608Metric, F.Cu at (124.6, 104.7)
- added C7: 47uF, Capacitor_SMD:C_0805_2012Metric, F.Cu at (126.4, 104.7)
- added C8: 4.7uF, Capacitor_SMD:C_0603_1608Metric, F.Cu at (179.4, 105.6)
- added D4: LED, Connector_PinSocket_2.54mm:PinSocket_1x02_P2.54mm_Vertical, F.Cu at (188.4, 90.4)
- added JP1: ~, Jumper:SolderJumper-2_P1.3mm_Open_RoundedPad1.0x1.5mm, F.Cu at (130.1, 113.5)
- added JP2: SolderJumper_2_Open, Jumper:SolderJumper-2_P1.3mm_Open_RoundedPad1.0x1.5mm, F.Cu at (129.6, 107.0)
- added JP3: SolderJumper_3_Open, Jumper:SolderJumper-3_P1.3mm_Open_RoundedPad1.0x1.5mm, F.Cu at (173.4, 81.3)
- added JP5: All or none, Jumper:SolderJumper-3_P1.3mm_Open_RoundedPad1.0x1.5mm, F.Cu at (171.4, 88.0)
- added L1: 22uH, Inductor_SMD:L_Wuerth_WE-TPC-3816, F.Cu at (121.4, 104.5)
- added L2: 10uH, Inductor_SMD:L_0603_1608Metric, F.Cu at (176.8, 107.7)
- added Q1: AO3401A, Package_TO_SOT_SMD:SOT-23, F.Cu at (172.8, 84.6)
- added Q2: AO3400A, Package_TO_SOT_SMD:SOT-23, F.Cu at (176.2, 84.6)
- added R11: 5.1M, Resistor_SMD:R_0603_1608Metric, F.Cu at (123.4, 114.5)
- added R12: 5.1M, Resistor_SMD:R_0603_1608Metric, F.Cu at (172.9, 123.3)
- added R13: 5.1M, Resistor_SMD:R_0603_1608Metric, F.Cu at (172.9, 121.8)
- added R14: 1k, Resistor_SMD:R_0603_1608Metric, F.Cu at (188.6, 94.8)
- added R15: 5.1M, Resistor_SMD:R_0603_1608Metric, F.Cu at (126.9, 113.0)
- added R16: 5.1M, Resistor_SMD:R_0603_1608Metric, F.Cu at (126.9, 114.5)
- added R17: 1M, Resistor_SMD:R_0603_1608Metric, F.Cu at (128.2, 116.0)
- added R18: 4.12M, Resistor_SMD:R_0603_1608Metric, F.Cu at (129.6, 109.0)
- added R19: 4.87M, Resistor_SMD:R_0603_1608Metric, F.Cu at (129.6, 110.5)
- added R23: 10M, Resistor_SMD:R_0603_1608Metric, F.Cu at (176.3, 87.3)
- added R4: 5.9M, Resistor_SMD:R_0603_1608Metric, F.Cu at (120.4, 110.0)
- added REF**: nothing, misc:nothing, F.Cu at (184.2, 126.7)
- added REF**: pg1425, pg1425:pg1425, F.Cu at (246.2, 156.3)
- added REF**: nothing, misc:nothing, F.Cu at (156.0, 65.0)
- added REF**: nothing, misc:nothing, F.Cu at (182.0, 75.2)
- added REF**: pg1425, pg1425:pg1425, F.Cu at (246.2, 139.3)
- added SC1: Solar_Cell, misc:KXOB25-05X3F, F.Cu at (116.5, 126.0)
- added SW3: SW_Push, Button_Switch_SMD:SW_SPST_B3U-1000P, F.Cu at (190.3, 88.1)
- added TP1: 3V3, TestPoint:TestPoint_THTPad_D1.0mm_Drill0.5mm, F.Cu at (182.0, 100.0)
- added TP2: GND, TestPoint:TestPoint_THTPad_D1.0mm_Drill0.5mm, F.Cu at (182.9, 96.7)
- added TP3: MOSI, TestPoint:TestPoint_THTPad_D1.0mm_Drill0.5mm, F.Cu at (174.9, 98.3)
- added TP4: DR, TestPoint:TestPoint_THTPad_D1.0mm_Drill0.5mm, F.Cu at (183.7, 98.6)
- added TP5: CS, TestPoint:TestPoint_THTPad_D1.0mm_Drill0.5mm, F.Cu at (184.9, 100.2)
- added TP6: MISO, TestPoint:TestPoint_THTPad_D1.0mm_Drill0.5mm, F.Cu at (176.9, 98.8)
- added TP7: SCLK, TestPoint:TestPoint_THTPad_D1.0mm_Drill0.5mm, F.Cu at (175.4, 100.4)
- added U2: XC6220B331MR, Package_TO_SOT_SMD:SOT-23-5, F.Cu at (169.3, 84.1)
- added U6: ~, Package_DFN_QFN:QFN-16-1EP_3x3mm_P0.5mm_EP1.7x1.7mm, F.Cu at (124.9, 109.2)
- added U7: MCP23S08, Package_SO:SOIC-18W_7.5x11.6mm_P1.27mm, F.Cu at (110.4, 98.3)
- C1: value 10nF -> 0.1uF
- C2: value 4.7uF -> Li Cap; footprint Capacitor_SMD:C_0603_1608Metric -> Capacitor_THT:CP_Radial_D13.0mm_P5.00mm
- C4: value 4.7uF -> 10nF
- C5: value 0.1uF -> 10nF
- D1: value RED -> D; footprint LED_SMD:LED_0805_2012Metric -> Diode_SMD:D_SOD-123
- H3: renamed from H9; footprint fusion:mount-magnet -> misc:m2-heat-insert-pad
- H4: renamed from H8; footprint fusion:mount-magnet -> misc:m2-heat-insert-pad
- H7: renamed from H17; footprint fusion:mount-magnet -> misc:m2-heat-insert-pad
- H8: renamed from H18; footprint fusion:mount-magnet -> misc:m2-heat-insert-pad
- J1: value tc2030 -> debug-port; footprint Connector:Tag-Connect_TC2030-IDC-NL_2x03_P1.27mm_Vertical -> misc:debug-port-single-side
- J5: value cirque-trackpad -> Conn_01x03_Female; footprint Connector_FFC-FPC:Hirose_FH12-12S-0.5SH_1x12-1MP_P0.50mm_Horizontal -> Connector_PinSocket_2.54mm:PinSocket_1x03_P2.54mm_Vertical
- K1, K11, K19, K24, K29, K6: footprint pg1232:pg1232-DSSN -> pg1232:pg1232-DCN
- K10, K15, K5: footprint pg1232:pg1232-DSSR -> pg1232:pg1232-DCN
- K12, K2, K22, K27, K32, K7: footprint pg1232:pg1232-DSSR -> pg1232:pg1232-DCR
- K13, K16, K17, K18, K21, K26, K3, K31, K36, K37, K38, K8: footprint pg1232:pg1232-DSS -> pg1232:pg1232-DC
- K14, K20, K25, K30, K4, K9: footprint pg1232:pg1232-DSSL -> pg1232:pg1232-DCL
- K23, K28, K33: footprint pg1232:pg1232-DSSL -> pg1232:pg1232-DCN
- R1: value 10k -> 4.12M
- R2: value 10k -> 10M
- R3: value 100k -> 22
- R5: value 5.1M -> 22
- R6: value 1k -> 5.1M
- R8: value 5.1M -> 5.1k
- R9: value 5.1k -> 1M
- SW1: value SW_Push -> SW_SPDT; footprint Button_Switch_SMD:SW_SPST_TL3342 -> Button_Switch_SMD:SW_SPDT_PCM12
- SW2: value SW_SPDT -> SW_Push; footprint Button_Switch_SMD:SW_SPDT_PCM12 -> Button_Switch_SMD:SW_SPST_TL3342
- U1: value holyiot-18010-no-underside -> ms88sf3-nrf52840; footprint mcu:holyiot-18010-no-underside -> mcu:ms88sf3
- U3: value BQ24075 -> TLV70237_SOT23-5; footprint Package_DFN_QFN:VQFN-16-1EP_3x3mm_P0.5mm_EP1.68x1.68mm_ThermalVias -> Package_TO_SOT_SMD:SOT-23-5
- moved C2 131.3 mm to (38.1, 89.8), turned to -112.5 degrees
- moved P1 106.3 mm to (142.3, 59.7), turned to 45 degrees
- moved R6 74.8 mm to (123.4, 113.0), turned to 0 degrees
- moved C3 61.8 mm to (117.4, 108.5)
- moved LCD1 61.6 mm to (118.0, 99.3)
- moved C4 59.0 mm to (120.4, 111.5)
- moved R2 57.5 mm to (117.4, 110.0), turned to 0 degrees
- moved R1 54.8 mm to (120.4, 108.5), turned to 0 degrees
- moved SW2 46.7 mm to (193.8, 108.8), turned to 22.5 degrees
- moved SW1 44.5 mm to (191.7, 63.9), turned to -157.5 degrees
- moved REF** 44.4 mm to (160.5, 130.5)
- moved C5 43.8 mm to (172.9, 120.3)
- moved D3 42.4 mm to (168.7, 128.1), turned to 90 degrees
- moved J5 31.5 mm to (191.6, 85.0), turned to 22.5 degrees
- moved R10 30.4 mm to (182.7, 101.8), turned to 0 degrees
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- renumbered D3 to D2, D2 to D3, H13 to H1, H2 to H10, H4 to H11, H2 to H12, H12 to H2, H11 to H5, H14 to H6, H4 to H9, REF** to P1, R12 to R20, R13 to R21, R14 to R22, U5 to U4, U8 to U5, U2 to U8
Connections:
- net R5 renamed /right/R1
- C1 pad 1: BAT_MEAS -> /right/SOLAR_OUT
- C2 pad 1: VBUS -> /left/CAP
- C2 pad 2: GND -> /left/GND
- C3 pad 1: GND -> /left/GND
- C3 pad 2: /power/VDDH -> /left/SOLAR
- C4 pad 1: BAT -> /left/GND
- C4 pad 2: GND -> Net-(C4-Pad2)
- C5 pad 1: /power/VDDH -> /right/BAT_MEAS
- D1 pad 2: /power/VDDH -> Net-(D1-Pad2)
- D2 pad 1: Net-(U1-Pad33) -> Net-(D2-Pad1)
- D2 pad 2: MAGNET -> /right/MAGNET
- D3 pad 2: +3V3 -> /right/3V3_nRF
- J1 pad 1: +3V3 -> GND
- J1 pad 2: SWD -> /right/3V3_nRF
- J1 pad 3: RST -> /right/SWD
- J1 pad 4: SWC -> /right/SWC
- J2 pad A4: VBUS -> /right/VBUS
- J2 pad A6: D+ -> /right/D+
- J2 pad A7: D- -> /right/D-
- J2 pad A9: VBUS -> /right/VBUS
- J2 pad B4: VBUS -> /right/VBUS
- J2 pad B6: D+ -> /right/D+
- J2 pad B7: D- -> /right/D-
- J2 pad B9: VBUS -> /right/VBUS
- J3 pad 1: /left/R3 -> /left/DISP_~{CS}
- J3 pad 10: unconnected-(J3-Pad10) -> /left/CAP
- J3 pad 12: /left/BAT -> /left/3V3
- J3 pad 2: /left/R2 -> /left/SCLK
- J3 pad 3: /left/R1 -> /left/MOSI
- J3 pad 4: /left/R0 -> /left/MISO
- J3 pad 5: /left/C4 -> /left/IO_~{CS}
- J3 pad 6: /left/C3 -> /left/IO_INT
- J3 pad 7: /left/C2 -> /left/C0
- J3 pad 8: /left/C1 -> unconnected-(J3-Pad8)
- J3 pad 9: /left/C0 -> /left/SOLAR_OUT
- J4 pad 1: BAT -> /right/3V3_nRF
- J4 pad 10: R1 -> /right/MOSI_DQ0
- J4 pad 11: R2 -> /right/SCLK
- J4 pad 12: R3 -> /right/DISP_~{CS}
- J4 pad 3: unconnected-(J4-Pad3) -> /right/BAT
- J4 pad 4: C0 -> /right/SOLAR_OUT
- J4 pad 5: C1 -> unconnected-(J4-Pad5)
- J4 pad 6: C2 -> /right/C0_LEFT
- J4 pad 7: C3 -> /right/IO_INT
- J4 pad 8: C4 -> /right/IO_~{CS}
- J4 pad 9: R0 -> /right/MISO_DQ1
- J4 pad MP: GND -> unconnected-(J4-PadMP)
- J5 pad 1: +3V3 -> /right/ENC_OUT
- J5 pad 2: GND -> /right/3V3_nRF
- J5 pad 3: unconnected-(J5-Pad3) -> GND
- K19 pad 1: R4 -> /right/R0
- K19 pad 2: C0 -> /right/C0
- K20 pad 1: R4 -> /right/R0
- K20 pad 2: C1 -> /right/C1
- K21 pad 1: R4 -> /right/R0
- K21 pad 2: C2 -> /right/C2
- K22 pad 1: R4 -> /right/R0
- K22 pad 2: C3 -> /right/C3
- K23 pad 1: R4 -> /right/R0
- K23 pad 2: C4 -> /right/C4
- K24 pad 2: C0 -> /right/C0
- K25 pad 2: C1 -> /right/C1
- K26 pad 2: C2 -> /right/C2
- K27 pad 2: C3 -> /right/C3
- K28 pad 2: C4 -> /right/C4
- K29 pad 1: R6 -> /right/R2
- K29 pad 2: C0 -> /right/C0
- K30 pad 1: R6 -> /right/R2
- K30 pad 2: C1 -> /right/C1
- K31 pad 1: R6 -> /right/R2
- K31 pad 2: C2 -> /right/C2
- K32 pad 1: R6 -> /right/R2
- K32 pad 2: C3 -> /right/C3
- K33 pad 1: R6 -> /right/R2
- K33 pad 2: C4 -> /right/C4
- K36 pad 1: R7 -> /right/R3
- K36 pad 2: C2 -> /right/C2
- K37 pad 1: R7 -> /right/R3
- K37 pad 2: C3 -> /right/C3
- K38 pad 1: R7 -> /right/R3
- K38 pad 2: C4 -> /right/C4
- LCD1 pad 1: DISP_~{CS} -> /left/DISP_~{CS}
- LCD1 pad 2: MOSI_DQ0 -> /left/MOSI
- LCD1 pad 3: SCLK -> /left/SCLK
- LCD1 pad 4: GND -> /left/GND
- LCD1 pad 5: +3V3 -> /left/3V3
- R1 pad 1: Net-(R1-Pad1) -> /left/SOLAR
- R1 pad 2: GND -> Net-(R1-Pad2)
- R10 pad 1: /power/VDDH -> /right/3V3_nRF
- R10 pad 2: MAGNET -> Net-(R10-Pad2)
- R2 pad 1: Net-(R2-Pad1) -> /left/GND
- R2 pad 2: GND -> Net-(R2-Pad2)
- R20 pad 1: ~{RED} -> /right/~{RED}
- R21 pad 1: ~{GREEN} -> /right/~{GREEN}
- R22 pad 1: ~{BLUE} -> /right/~{BLUE}
- R3 pad 1: +3V3 -> Net-(D1-Pad1)
- R3 pad 2: Net-(R3-Pad2) -> /right/BAT
- R5 pad 1: BAT -> Net-(D1-Pad1)
- R5 pad 2: BAT_MEAS -> /right/BAT
- R6 pad 1: Net-(R6-Pad1) -> /left/GND
- R6 pad 2: Net-(D1-Pad1) -> Net-(R11-Pad1)
- R8 pad 1: BAT_MEAS -> GND
- R8 pad 2: GND -> Net-(J2-PadB5)
- R9 pad 1: GND -> /right/SOLAR_OUT
- R9 pad 2: Net-(J2-PadB5) -> /right/MAGNET
- SW1 pad 1: RST -> /right/MAGNET
- SW1 pad 2: GND -> Net-(JP3-Pad2)
- SW2 pad 1: MAGNET -> /right/RST
- SW2 pad 2: Net-(SW2-Pad2) -> GND
- U1 pad 10: TP_~{CS} -> /right/~{RED}
- U1 pad 11: BAT_MEAS -> /right/~{GREEN}
- U1 pad 12: MISO_DQ1 -> /right/~{BLUE}
- U1 pad 13: MOSI_DQ0 -> unconnected-(U1-Pad13)
- U1 pad 2: C0 -> unconnected-(U1-Pad2)
- U1 pad 3: C1 -> unconnected-(U1-Pad3)
- U1 pad 32: GND -> /right/VDDH
- U1 pad 33: Net-(U1-Pad33) -> Net-(L2-Pad1)
- U1 pad 34: C4 -> GND
- U1 pad 35: R0 -> /right/VBUS
- U1 pad 36: R1 -> /right/D-
- U1 pad 37: SWD -> /right/D+
- U1 pad 38: SWC -> /right/DISP_~{CS}
- U1 pad 39: R2 -> /right/IO_~{CS}
- U1 pad 4: C2 -> unconnected-(U1-Pad4)
- U1 pad 40: R3 -> /right/IO_INT
- U1 pad 41: R4 -> /right/C0_LEFT
- U1 pad 43: TP_DR -> /right/R0
- U1 pad 44: GND -> /right/C4
- U1 pad 45: D+ -> /right/C3
- U1 pad 46: D- -> /right/C2
- U1 pad 47: VBUS -> /right/C1
- U1 pad 48: RST -> /right/C0
- U1 pad 49: ~{BLUE} -> /right/SWC
- U1 pad 5: R7 -> unconnected-(U1-Pad5)
- U1 pad 50: ~{GREEN} -> /right/SWD
- U1 pad 51: ~{RED} -> unconnected-(U1-Pad51)
- U1 pad 52: FLASH_~{CS} -> unconnected-(U1-Pad52)
- U1 pad 53: R6 -> unconnected-(U1-Pad53)
- U1 pad 54: SCLK -> unconnected-(U1-Pad54)
- U1 pad 55: +3V3 -> unconnected-(U1-Pad55)
- U1 pad 6: C3 -> unconnected-(U1-Pad6)
- U1 pad 7: DISP_~{CS} -> unconnected-(U1-Pad7)
- U1 pad 9: unconnected-(U1-Pad9) -> /right/R2
- U3 pad 1: Net-(R1-Pad1) -> /right/VBUS
- U3 pad 2: BAT -> GND
- U3 pad 3: BAT -> /right/VBUS
- U3 pad 4: GND -> unconnected-(U3-Pad4)
- U3 pad 5: GND -> Net-(D1-Pad2)
- U4 pad 1: /power/VDDH -> /right/SOLAR_OUT
- U4 pad 2: MAGNET -> /right/MAGNET
- U5 pad 1: D- -> /right/D-
- U5 pad 3: D+ -> /right/D+
- U5 pad 4: D+ -> /right/D+
- U5 pad 5: VBUS -> /right/VBUS
- U5 pad 6: D- -> /right/D-
- U8 pad 1: FLASH_~{CS} -> /right/FLASH_~{CS}
- U8 pad 2: MISO_DQ1 -> /right/MISO_DQ1
- U8 pad 3: Net-(R3-Pad2) -> Net-(R10-Pad2)
- U8 pad 5: MOSI_DQ0 -> /right/MOSI_DQ0
- U8 pad 6: SCLK -> /right/SCLK
- U8 pad 7: Net-(R3-Pad2) -> Net-(R10-Pad2)
- U8 pad 8: +3V3 -> /right/3V3_nRF
Routing:
- net C0: track 211.7 -> 0.00 mm, vias 6 -> 0
- net C2: track 197.6 -> 0.00 mm, vias 4 -> 0
- net R7: track 193.8 -> 0.00 mm
- net C1: track 190.4 -> 0.00 mm, vias 4 -> 0
- net /right/C0: track 0.00 -> 187.6 mm, vias 0 -> 4
- net /right/C2: track 0.00 -> 175.5 mm, vias 0 -> 2
- net C3: track 168.5 -> 0.00 mm, vias 4 -> 0
- net /right/C3: track 0.00 -> 150.3 mm, vias 0 -> 2
- net /right/C1: track 0.00 -> 145.9 mm, vias 0 -> 4
- net C4: track 133.1 -> 0.00 mm, vias 2 -> 0
- net R4: track 132.4 -> 0.00 mm, vias 1 -> 0
- net /right/C4: track 0.00 -> 128.4 mm, vias 0 -> 2
- net /right/R2: track 0.00 -> 126.0 mm, vias 0 -> 1
- net R6: track 125.9 -> 0.00 mm, vias 1 -> 0
- net /right/R0: track 0.00 -> 122.8 mm, vias 0 -> 1
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- added copper zone on B.Cu, net /left/GND
- added copper zone on F.Cu, net /left/GND
Other:
- board size 280 x 97 mm -> 271.7 x 89.5 mm
