File: trackpad-8520.kicad_sch (KiCad schematic)
At the start: 6 parts, among them J5 Conn_02x10_Odd_Even_MountingP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, U6 MIC5365-2.8YC5, U7 4050

Commit message: Hydrogen.PCB
- add Adafruit CAD files for Sharp display
- convert to all 3D printed mechanical parts
- update part dimensions to lowest estimate
Parts:
- J5: now left out of the parts list
Changed lines of the file:
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@@
   )
   (symbol (lib_id "Connector_Generic_MountingPin:Conn_02x10_Odd_Even_MountingPin") (at 50.8 165.1 0) (unit 1)
-    (in_bom yes) (on_board yes)
+    (in_bom no) (on_board yes)
     (property "Reference" "J5" (id 0) (at 52.07 144.6234 0))
     (property "Value" "Conn_02x10_Odd_Even_MountingPin" (id 1) (at 52.07 146.1285 0))
