File: fusion.kicad_sch (KiCad schematic)
At the start: 46 parts, among them J1 debug-port, J3 Conn_01x12_MountingPin, J4 Conn_01x12_MountingPin, J5 cirque-trackpad, K19 diode-choc, K20 diode-choc, K21 diode-choc, K22 diode-choc, K23 diode-choc, K24 diode-choc, K25 diode-choc, K26 diode-choc, K27 diode-choc, K28 diode-choc, K29 diode-choc, K30 diode-choc, K31 diode-choc, K32 diode-choc, K33 diode-choc, K34 diode-choc, K35 diode-choc, K36 diode-choc, K37 diode-choc, K38 diode-choc, SW1 SW_Push, U1 holyiot-18010-no-underside, U2 MT25QL128ABA1ESE

Commit message: new version
Parts:
- removed J1: debug-port, misc:debug-port-single-side, symbol misc:debug-port
- removed JP4: SolderJumper_2_Open, Jumper:SolderJumper-2_P1.3mm_Open_RoundedPad1.0x1.5mm, symbol Jumper:SolderJumper_2_Open
- added D3: D_Small, Diode_SMD:D_SOD-123, symbol Device:D_Small
- added J1: tc2030, Connector:Tag-Connect_TC2030-IDC-NL_2x03_P1.27mm_Vertical, symbol misc:tc2030
Connections:
- net +3V3: now also J1.1 (VCC)
- net GND: now also J1.5 (GND)
- net MAGNET: now also D3.2 (A)
- net RST: now also J1.3 (~{RST})
- net SWC: now also J1.4 (SWC)
- net SWD: now also J1.2 (SWD)
- net at U1.33 ([L]_P0.10): now also D3.1 (K)
- no-connect marks 4 -> 5

Commit message: backup & remove useless things
Parts:
- removed C1: 10nF, Capacitor_SMD:C_0603_1608Metric, symbol Device:C
- removed D2: LED_RABG, LED_SMD:LED_ASMB-KTF0-0A306, symbol Device:LED_RABG
- removed D3: D_Small, Diode_SMD:D_SOD-123, symbol Device:D_Small
- removed H11, H12: hinge-big, fusion:hinge2, symbol Mechanical:MountingHole
- removed H13, H14: hinge-small, fusion:hinge1, symbol Mechanical:MountingHole
- removed H17, H18, H8, H9: mount-magnet, fusion:mount-magnet, symbol Mechanical:MountingHole
- removed H20: bat-shell, fusion:bat-shell-small, symbol Mechanical:MountingHole
- removed J1: tc2030, Connector:Tag-Connect_TC2030-IDC-NL_2x03_P1.27mm_Vertical, symbol misc:tc2030
- removed J5: cirque-trackpad, Connector_FFC-FPC:Hirose_FH12-12S-0.5SH_1x12-1MP_P0.50mm_Horizontal, symbol misc:cirque-trackpad
- removed K19, K24, K29, K34, K35: diode-choc, pg1232:pg1232-DSSN, symbol diode-choc:diode-choc
- removed K20, K23, K25, K28, K30, K33: diode-choc, pg1232:pg1232-DSSL, symbol diode-choc:diode-choc
- removed K21, K26, K31, K36, K37, K38: diode-choc, pg1232:pg1232-DSS, symbol diode-choc:diode-choc
- removed K22, K27, K32: diode-choc, pg1232:pg1232-DSSR, symbol diode-choc:diode-choc
- removed LCD1: adafruit-sharp-memory-display-no-useless, display:adafruit-sharp-memory-display-1.3in-no-mounting-no-useless, symbol display:adafruit-sharp-memory-display-no-useless
- removed R12: 1.2k, Resistor_SMD:R_0603_1608Metric, symbol Device:R
- removed R13: 1.5k, Resistor_SMD:R_0603_1608Metric, symbol Device:R
- removed R14: 1k, Resistor_SMD:R_0603_1608Metric, symbol Device:R
- removed R3: 100k, Resistor_SMD:R_0603_1608Metric, symbol Device:R
- removed R5, R8: 5.1M, Resistor_SMD:R_0603_1608Metric, symbol Device:R
- removed SW1: SW_Push, Button_Switch_SMD:SW_SPST_TL3342, symbol Switch:SW_Push
- removed U1: holyiot-18010-no-underside, mcu:holyiot-18010-no-underside, symbol mcu:holyiot-18010-no-underside
- removed U2: MT25QL128ABA1ESE, Package_SO:SOIC-8_5.23x5.23mm_P1.27mm, symbol ic:MT25QL128ABA1ESE
Connections:
- net left/C2 is gone; now on net left/C0: J3.7 (Pin_7)
- net left/C0: no longer J3.9 (Pin_9)
- net right/BAT: now reaches J4.3 (Pin_3)
- net left/CAP: now reaches J3.10 (Pin_10)
- net BAT renamed right/3V3
- net C0 renamed right/SOLAR_OUT
- net C1: no longer names the net of J4.5 (Pin_5)
- net C2 renamed right/C0_LEFT
- net C3 renamed right/IO_INT
- net C4 renamed right/IO_~{CS}
- net GND: no longer names the net of J4.MP (MountPin)
- net GND: no longer J4.2 (Pin_2)
- net R0 renamed right/MISO_DQ1
- net R1 renamed right/MOSI_DQ0
- net R2 renamed right/SCLK
- net R3 renamed right/DISP_~{CS}
- net left/BAT renamed left/3V3
- net left/C1: no longer names the net of J3.8 (Pin_8)
- net left/C3 renamed left/IO_INT
- net left/C4 renamed left/IO_~{CS}
- net left/R0 renamed left/MISO
- net left/R1 renamed left/MOSI
- net left/R2 renamed left/SCLK
- net left/R3 renamed left/DISP_~{CS}
- new net left/SOLAR_OUT: J3.9 (Pin_9)
- new net right/GND: J4.2 (Pin_2)
- no-connect marks 5 -> 0
Other:
- removed sheet power
- added sheet right (right.kicad_sch)
- sheet left ports: added 3V3, CAP, DISP_~{CS}, IO_INT, IO_~{CS}, MISO, MOSI, SCLK, SOLAR_OUT; removed BAT, C1, C2, C3, C4, R0, R1, R2, R3
- moved on the sheet: J3, J4
